Commit message: Update cartpole.urdf

File: examples/assets/cartpole.urdf (robot description, URDF)
Before this commit: robot cartpole, 4 links, 3 joints
Joints:
- joint pivot: limit lower=-3.4028234663852886e+38 upper=3.4028234663852886e+38 effort=500.0 velocity=10.0 -> lower=-1000000000 upper=1000000000 effort=500.0 velocity=10.0
